File: MP3Part1/iCE40UP5Kdev/iCE40UP5Kdev.kicad_pcb (KiCad board)
At the start: 2 copper layers, 35.3 x 52.8 mm, 51 parts, among them J1 USB4105-GF-A, J2 Left, J3 Right, U1 W25Q32JV, U2 MIC5365-1-2YD5, U3 MIC5318-3-3YD5, U4 ICE40UP5K-SG48ITR, X1 IQXO-791

Commit message: reorganized loose files for MP3
Parts:
- moved C12 6.39 mm to (36.3, 34.6)
- moved C11 6.39 mm to (39.5, 40.9), turned to 0 degrees
- moved D4 3.90 mm to (42.6, 40.9), turned to 0 degrees
- moved R5 2.06 mm to (41.4, 29.5)
- moved S1 1.60 mm to (41.5, 24.3)
- moved C14 0.55 mm to (38.9, 34.7)
- moved C15 0.55 mm to (40.5, 34.7)
Routing:
- net Net-(D4-K): track 12.3 -> 5.91 mm, vias 2 -> 0
- net GND: track 87.6 -> 92.2 mm, vias 25 -> 27
- net /IOT_42b: track 48.0 -> 43.8 mm
- net /IOT_43a: track 43.8 -> 39.6 mm
- net +3V3: track 183.0 -> 186.0 mm, vias 9 -> 10
- net Net-(U4-~{CRESET}): track 36.5 -> 38.9 mm
- net /IOT_46b_G0: track 39.9 -> 41.1 mm
- net /RGB0: track 53.2 -> 54.2 mm
- net /IOT_36b: track 18.3 -> 19.2 mm
- net Net-(U1-DO/IO1): track 7.92 -> 7.29 mm
- net Net-(U4-VCCPLL): track 7.64 -> 8.20 mm
- net Net-(U4-IOB_25b_G3): track 7.56 -> 8.07 mm
- net (no net): vias 2 -> 0
